File: KiCAD/Plasma_Pilot4/Plasma_Pilot4.sch (KiCad schematic (older format))
At the start: 80 parts, among them IC1 ATTINY861A-S, P1 CONN_02X03, P2 CONN_01X02, P3 CONN_01X02, P4 CONN_01X02, P5 CONN_01X02, P6 CONN_01X02, P7 CONN_01X03, P8 CONN_01X03, Q1 BSS138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

Commit message: Added new transformer fixed code to work on CT600 plasma cutter
Parts:
- removed R19: 1000, t_passive_smd:res_0805, symbol Plasma_Pilot4-rescue:Rx-Plasma_Pilot4-rescue-Plasma_Pilot4-rescue
- removed R21: 10K, t_passive_smd:res_0603, symbol t_Devices:Res6
- removed T1: EP10_GDT, t_coilcraft:EP10_SMT, symbol t_Coilcraft:EP10_GDT
- added R19: 1.0K, t_passive_smd:res_0603, symbol t_Devices:Res6
- added T?: EP10_GDT_2, t_coilcraft:EP10_SMT, symbol t_Coilcraft:EP10_GDT_2
- C10: value 0.1uF -> 0.022uF
- C7: value 0.1uF -> 1000pF
- Q2, Q4: value BSS138 -> BSS131
- R11, R12: value Res6 -> 6.8K
- R13: value 220 -> 1.0K
- R20: value 10K -> 100; footprint t_passive_smd:res_0603 -> t_passive_smd:res_0805
- R23: value Res6 -> 392K
- R24: value Res6 -> 50K
- R25: value Res6 -> 10K
- R26: value Res6 -> 1.0K
Connections:
- net GND: now also R20.1; no longer R20.2
- net at C3.1, Q2.3 (D), Q4.3 (D): now also T?.8 (P2)
- net at C1.1, R22.1: now also T?.5 (P1)
- net at C7.1, R8.1: now also D3.1 (A); no longer D3.2 (K)
- net at C10.2, Q3.3 (E), TP2.1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: no longer C7.2, P5.2 (P2), R9.2
- net at P5.1 (P1), R8.2, R9.1: no longer Q3.1 (G), TP1.1
- net at P6.1 (P1), TP5.1: now also R20.2, R19.2
- net at U3.3 (+): now also R19.1; no longer R20.1
- new net: C7.2, P5.2 (P2), R9.2, T?.4 (S2)
- new net: Q3.1 (G), TP1.1
- new net: D3.2 (K), T?.1 (S1)
Other:
- note added: "0.1 Ohm Sense\nResistor goes here"
- note added: "275 KHz 1.0us \nPulse width"
- note added: "36:24"
- note added: "CT520 - START Connects Trigger/Foot Pedal switch\nDon't connect to the +24V side of the switch! \n(Con 11 Red?) \nAbout 10V when switch is open , \n+24V when trigger is pressed\n\nCT6000 no voltage when open, +24V when \nTrigger Pressed (Red Wire)"
- note added: "CT6000 Open Circuit Voltage -280V\nNeed another 100K in series"
- note added: "Gate"
- note added: "Primary L 250uH\nGluing with JB Weld \ncauses slight gap"
- note added: "R17:\n1.0K on CT6000\n15K on CT520D"
- note added: "Source"
- note removed: "0.2 Ohm Sense\nResistor goes here"
- note removed: "200 KHz 1.7us \nPulse width"
- note removed: "CT520 - START Connects Trigger/Foot Pedal switch\nDon't connect to the +24V side of the switch! \n(Con 11 Red?) Open when not in use, +24V\nwhen trigger is pressed"
- moved on the sheet: C17, R20
